File: Hardware/RGB_board/RGB_board.kicad_sch (KiCad schematic)
At the start: 33 parts, among them J10 Conn_01x02, J2 Screw_Terminal_01x02, J3 Screw_Terminal_01x04, J4 Screw_Terminal_01x02, J5 Conn_01x02, J6 Conn_01x02, J7 Conn_01x02, J8 Conn_01x04, J9 Conn_01x04, Q1 Si1308EDL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

Commit message: Refactor code structure for improved readability and maintainability
Parts:
- removed J10, J5, J6, J7: Conn_01x02, Connector_PinSocket_2.54mm:PinSocket_1x02_P2.54mm_Vertical, symbol Connector_Generic:Conn_01x02
- removed J2, J4: Screw_Terminal_01x02, TerminalBlock_Phoenix:TerminalBlock_Phoenix_PT-1,5-2-3.5-H_1x02_P3.50mm_Horizontal, symbol Connector:Screw_Terminal_01x02
- removed J3: Screw_Terminal_01x04, TerminalBlock_Phoenix:TerminalBlock_Phoenix_PT-1,5-4-3.5-H_1x04_P3.50mm_Horizontal, symbol Connector:Screw_Terminal_01x04
- removed J8: Conn_01x04, Connector_PinSocket_2.54mm:PinSocket_1x04_P2.54mm_Vertical, symbol Connector_Generic:Conn_01x04
- removed J9: Conn_01x04, Connector:FanPinHeader_1x04_P2.54mm_Vertical, symbol Connector_Generic:Conn_01x04
- removed Q4: Si1308EDL, Package_TO_SOT_SMD:SOT-323_SC-70, symbol Transistor_FET:Si1308EDL
- removed R10, R11, R9: 1k5, Resistor_SMD:R_0805_2012Metric, symbol Device:R
- removed SW1: SW_SPDT, aa_MyParts:SW_200MSP1T1B2M6QE_EWI, symbol aa_MyParts:SW_200MSP1T1B2M6QE_1
- removed SW2: SW_Push_SPST, aa_MyParts:SW_800AWSP9M6QE, symbol Switch:SW_800AWSP9M6QE
- removed U1, U2, U3: VO615A-2X009T, Package_DIP:DIP-4_W8.89mm_SMDSocket_LongPads, symbol Isolator:VO615A-2
- added C1, C2: 10uF, Capacitor_SMD:C_0805_2012Metric, symbol Device:C
- added C3: 100nF, Capacitor_SMD:C_0805_2012Metric, symbol Device:C
- added C4, C5: 22uF, Capacitor_SMD:C_0805_2012Metric, symbol Device:C
- added D1: CDBC540-G, Diode_SMD:D_SMC, symbol Device:D
- added J1: Conn_01x11, symbol Connector_Generic:Conn_01x11
- added J2, J3: Conn_01x04, symbol Connector_Generic:Conn_01x04
- added U1: TPS563200, Package_TO_SOT_SMD:SOT-23-6, symbol Regulator_Switching:TPS563200
- R1, R3, R5: value 15k -> 100R
- R7: value 1k5 -> 56k2; LCSC Part # C4310 -> C17475
- R8: value 680k -> 10k; LCSC Part # C17797 -> C17475
Connections:
- net FAN_control is gone; now on an unnamed net: R7.1
- net GND_ISO is gone; now on net GND: Q1.2 (S), Q2.2 (S), Q3.2 (S), R2.1, R4.1, R6.1
- net LED_opt_blue is gone; now on net LED_control_blue: R5.1
- net LED_opt_green is gone; now on net LED_control_green: R3.1
- net LED_opt_red is gone; now on net LED_control_red: R1.1
- net +5V: now also R7.2, C3.1, C4.1, C5.1, J2.3 (Pin_3), U1.2 (SW)
- net GND: now also C1.2, C2.2, C4.2, C5.2, J1.11 (Pin_11), J2.2 (Pin_2), J2.4 (Pin_4), U1.1 (GND)
- net LED_blue_-: now also J3.4 (Pin_4)
- net LED_control_blue: now also J1.8 (Pin_8)
- net LED_control_green: now also J1.7 (Pin_7)
- net LED_control_red: now also J1.6 (Pin_6)
- net LED_green_-: now also J3.3 (Pin_3)
- net LED_red_-: now also J3.2 (Pin_2)
- net at R8.2: now also U1.4 (VFB); no longer R7.2
- new net: C3.2, U1.6 (VBST)
- new net: D1.2 (A), J2.1 (Pin_1)
- new net +12V: C1.1, C2.1, D1.1 (K), J3.1 (Pin_1), U1.3 (VIN), U1.5 (EN)
- new net 3V: J1.10 (Pin_10)
- new net A4: J1.9 (Pin_9)
- new net BOOT: J1.2 (Pin_2)
- new net DEBUG: J1.3 (Pin_3)
- new net RESET: J1.1 (Pin_1)
- new net RXI: J1.5 (Pin_5)
- new net TXO: J1.4 (Pin_4)
Other:
- note added: "5V Supply for LED Matrix"
- note added: "A1"
- note added: "A2"
- note added: "A3"
- note removed: "0.6mA"
- note removed: "1mA"
- note removed: "Fan External"
- note removed: "LCD+FAN"
- note removed: "Reset"
- note removed: "Temp Sensor External"
- title: 3D Printer Pi Hat -> Matrix LED RGB HAT
- moved on the sheet: Q1, Q3, R1, R2, R3, R4, R5, R6

Commit message: große fortschritte, mockup bereit
Parts:
- removed H1, H2, H3, H4: MountingHole, MountingHole:MountingHole_3.2mm_M3_DIN965, symbol Mechanical:MountingHole
- added H1: +5V_Screw, aa_MyParts:H_3.2mm_M3_Pad_7mm, symbol Mechanical:MountingHole_Pad
- added H2: GND_Screw, aa_MyParts:H_3.2mm_M3_Pad_7mm, symbol Mechanical:MountingHole_Pad
- added L1: 3.3uH, 6A, Inductor_SMD:L_Bourns_SRP7028A_7.3x6.6mm, symbol Device:L
- J1: footprint (none) -> aa_MyParts:J_FM11x2_2.5476341-311LF
- J2, J3: footprint (none) -> aa_MyParts:T_4_PhoenixContact_LPT_5_4-H-1x04_Horizontal
Connections:
- net +12V: now also J3.4 (Pin_4); no longer J3.1 (Pin_1)
- net +5V: now also J2.2 (Pin_2), H1.1, L1.2; no longer C3.1, J2.3 (Pin_3), U1.2 (SW)
- net GND: now also J2.1 (Pin_1), J2.3 (Pin_3), H2.1; no longer J2.2 (Pin_2), J2.4 (Pin_4)
- net LED_blue_-: now also J3.1 (Pin_1); no longer J3.4 (Pin_4)
- net LED_green_-: now also J3.2 (Pin_2); no longer J3.3 (Pin_3)
- net LED_red_-: now also J3.3 (Pin_3); no longer J3.2 (Pin_2)
- net at D1.2 (A): now also J2.4 (Pin_4); no longer J2.1 (Pin_1)
- new net: C3.1, L1.1, U1.2 (SW)
Other:
- moved on the sheet: C4, C5, R7, R8
